Commit message: add indicator link

File: ipa_canopen_test/urdf/elmo_test_rig.urdf.xacro (robot description, xacro)
@@ -8,4 +8,5 @@
   <property name="plate_height" value="0.01" />
   <property name="plate_radius" value="0.03" />
+  <property name="indicator_height" value="0.001" />
   <link name="base_link" >
     <visual>
@@ -51,3 +52,26 @@
     </xacro:cylinder_inertial>
   </link>
+  <joint name="indicator_joint" type="fixed">
+    <parent link="plate_link" />
+    <child link = "indicator_link" />
+    <origin xyz="0.0 0.0 ${plate_height}" rpy="0 0 0" />
+  </joint>
+  <link name="indicator_link" >
+    <visual>
+      <origin xyz="${plate_radius/2} 0.0 ${indicator_height/2}" rpy="0 0 0" />
+      <geometry>
+        <box size="${plate_radius} ${indicator_height} ${indicator_height}" />
+      </geometry>
+      <material name="IPA/Orange"/>
+    </visual>
+    <collision>
+      <origin xyz="${plate_radius/2} 0.0 ${indicator_height/2}" rpy="0 0 0" />
+      <geometry>
+        <box size="${plate_radius} ${indicator_height} ${indicator_height}" />
+      </geometry>
+    </collision>
+    <xacro:box_inertial x="${plate_radius}" y="${indicator_height}" z="${indicator_height}" mass="0.050">
+      <origin xyz="${plate_radius/2} 0.0 ${indicator_height/2}" rpy="0 0 0" />
+    </xacro:box_inertial>
+  </link>
 </robot>

Commit message: add 2dof test rig urdf

File: ipa_canopen_test/urdf/elmo_test_rig.urdf.xacro (robot description, xacro)
@@ -10,77 +10,84 @@
   <property name="plate_radius" value="0.03" />
   <property name="indicator_height" value="0.001" />
-  <link name="base_link" >
-    <visual>
-      <origin xyz="0.0 0.0 ${base_height/2}" rpy="0 0 0" />
-      <geometry>
-        <cylinder length="${base_height}" radius="${base_radius}" />
-      </geometry>
-    </visual>
-    <collision>
-      <origin xyz="0.0 0.0 ${base_height/2}" rpy="0 0 0" />
-      <geometry>
-        <cylinder length="${base_height}" radius="${base_radius}" />
-      </geometry>
-    </collision>
-    <xacro:cylinder_inertial radius="${base_radius}" length="${base_height}" mass="0.100">
-      <origin xyz="0.0 0.0 ${base_height/2}" rpy="0 0 0" />
-    </xacro:cylinder_inertial>
-  </link>
-  <joint name="plate_joint" type="revolute">
-    <parent link="base_link" />
-    <child link = "plate_link" />
-    <origin xyz="0.0 0.0 ${base_height}" rpy="0.0 0.0 0.0" />
-    <axis xyz="0 0 1" />
-    <limit lower="${-M_PI}" upper="${M_PI}" effort="10.0" velocity="3.15"/>
-    <dynamics damping="0.0" friction="0.0"/>
-  </joint>
-  <link name="plate_link" >
-    <visual>
-      <origin xyz="0.0 0.0 ${plate_height/2}" rpy="0 0 0" />
-      <geometry>
-        <cylinder length="${plate_height}" radius="${plate_radius}" />
-      </geometry>
-      <material name="IPA/Blue"/>
-    </visual>
-    <collision>
-      <origin xyz="0.0 0.0 ${plate_height/2}" rpy="0 0 0" />
-      <geometry>
-        <cylinder length="${plate_height}" radius="${plate_radius}" />
-      </geometry>
-    </collision>
-    <xacro:cylinder_inertial radius="${plate_radius}" length="${plate_height}" mass="0.100">
-      <origin xyz="0.0 0.0 ${plate_height/2}" rpy="0 0 0" />
-    </xacro:cylinder_inertial>
-  </link>
-  <joint name="indicator_joint" type="fixed">
-    <parent link="plate_link" />
-    <child link = "indicator_link" />
-    <origin xyz="0.0 0.0 ${plate_height}" rpy="0 0 0" />
-  </joint>
-  <link name="indicator_link" >
-    <visual>
-      <origin xyz="${plate_radius/2} 0.0 ${indicator_height/2}" rpy="0 0 0" />
-      <geometry>
-        <box size="${plate_radius} ${indicator_height} ${indicator_height}" />
-      </geometry>
-      <material name="IPA/Orange"/>
-    </visual>
-    <collision>
-      <origin xyz="${plate_radius/2} 0.0 ${indicator_height/2}" rpy="0 0 0" />
-      <geometry>
-        <box size="${plate_radius} ${indicator_height} ${indicator_height}" />
-      </geometry>
-    </collision>
-    <xacro:box_inertial x="${plate_radius}" y="${indicator_height}" z="${indicator_height}" mass="0.050">
-      <origin xyz="${plate_radius/2} 0.0 ${indicator_height/2}" rpy="0 0 0" />
-    </xacro:box_inertial>
-  </link>
-  <!-- extensions -->
-  <xacro:torso_transmission name="plate" />
-  <gazebo>
-    <plugin name="ros_control" filename="libgazebo_ros_control.so">
-      <!--robotNamespace>/</robotNamespace-->
-      <!--robotSimType>gazebo_ros_control/DefaultRobotHWSim</robotSimType-->
-    </plugin>
-  </gazebo>
+  <xacro:macro name="elmo_test_rig" params="prefix parent *origin">
+    <joint name="${prefix}base_joint" type="fixed">
+      <parent link="${parent}" />
+      <child link = "${prefix}base_link" />
+      <insert_block name="origin" />
+    </joint>
+    <link name="${prefix}base_link" >
+      <visual>
+        <origin xyz="0.0 0.0 ${base_height/2}" rpy="0 0 0" />
+        <geometry>
+          <cylinder length="${base_height}" radius="${base_radius}" />
+        </geometry>
+      </visual>
+      <collision>
+        <origin xyz="0.0 0.0 ${base_height/2}" rpy="0 0 0" />
+        <geometry>
+          <cylinder length="${base_height}" radius="${base_radius}" />
+        </geometry>
+      </collision>
+      <xacro:cylinder_inertial radius="${base_radius}" length="${base_height}" mass="0.100">
+        <origin xyz="0.0 0.0 ${base_height/2}" rpy="0 0 0" />
+      </xacro:cylinder_inertial>
+    </link>
+    <joint name="${prefix}plate_joint" type="revolute">
+      <parent link="${prefix}base_link" />
+      <child link = "${prefix}plate_link" />
+      <origin xyz="0.0 0.0 ${base_height}" rpy="0.0 0.0 0.0" />
+      <axis xyz="0 0 1" />
+      <limit lower="${-M_PI}" upper="${M_PI}" effort="10.0" velocity="3.15"/>
+      <dynamics damping="0.0" friction="0.0"/>
+    </joint>
+    <link name="${prefix}plate_link" >
+      <visual>
+        <origin xyz="0.0 0.0 ${plate_height/2}" rpy="0 0 0" />
+        <geometry>
+          <cylinder length="${plate_height}" radius="${plate_radius}" />
+        </geometry>
+        <material name="IPA/Blue"/>
+      </visual>
+      <collision>
+        <origin xyz="0.0 0.0 ${plate_height/2}" rpy="0 0 0" />
+        <geometry>
+          <cylinder length="${plate_height}" radius="${plate_radius}" />
+        </geometry>
+      </collision>
+      <xacro:cylinder_inertial radius="${plate_radius}" length="${plate_height}" mass="0.100">
+        <origin xyz="0.0 0.0 ${plate_height/2}" rpy="0 0 0" />
+      </xacro:cylinder_inertial>
+    </link>
+    <joint name="${prefix}indicator_joint" type="fixed">
+      <parent link="${prefix}plate_link" />
+      <child link = "${prefix}indicator_link" />
+      <origin xyz="0.0 0.0 ${plate_height}" rpy="0 0 0" />
+    </joint>
+    <link name="${prefix}indicator_link" >
+      <visual>
+        <origin xyz="${plate_radius/2} 0.0 ${indicator_height/2}" rpy="0 0 0" />
+        <geometry>
+          <box size="${plate_radius} ${indicator_height} ${indicator_height}" />
+        </geometry>
+        <material name="IPA/Orange"/>
+      </visual>
+      <collision>
+        <origin xyz="${plate_radius/2} 0.0 ${indicator_height/2}" rpy="0 0 0" />
+        <geometry>
+          <box size="${plate_radius} ${indicator_height} ${indicator_height}" />
+        </geometry>
+      </collision>
+      <xacro:box_inertial x="${plate_radius}" y="${indicator_height}" z="${indicator_height}" mass="0.050">
+        <origin xyz="${plate_radius/2} 0.0 ${indicator_height/2}" rpy="0 0 0" />
+      </xacro:box_inertial>
+    </link>
+    <!-- extensions -->
+    <xacro:torso_transmission name="${prefix}plate" />
+    <gazebo>
+      <plugin name="ros_control" filename="libgazebo_ros_control.so">
+        <!--robotNamespace>/</robotNamespace-->
+        <!--robotSimType>gazebo_ros_control/DefaultRobotHWSim</robotSimType-->
+      </plugin>
+    </gazebo>
+  </xacro:macro>
 </robot>
