Commit message: introduce robot arg

File: ipa_canopen_test/urdf/rig12.urdf.xacro (robot description, xacro)
@@ -1,9 +1,12 @@
 <?xml version="1.0"?>
 <robot xmlns:xacro="http://www.ros.org/wiki/xacro"
-       name="elmo_test_rig" >
+       name="rig12" >
   <xacro:include filename="$(find ipa_canopen_test)/urdf/elmo_test_rig.urdf.xacro" />
   <link name="world" />"
-  <xacro:elmo_test_rig prefix="" parent="world">
-    <origin xyz="0.0 0.0 0.0" rpy="0 0 0" />
+  <xacro:elmo_test_rig prefix="rig1_" parent="world">
+    <origin xyz="0.0 0.2 0.0" rpy="0 0 0" />
+  </xacro:elmo_test_rig>
+  <xacro:elmo_test_rig prefix="rig2_" parent="world">
+    <origin xyz="0.0 -0.2 0.0" rpy="0 0 0" />
   </xacro:elmo_test_rig>
   <gazebo>

File: ipa_canopen_test/urdf/rig1_rig2.urdf.xacro (robot description, xacro)
@@ -1,5 +1,5 @@
 <?xml version="1.0"?>
 <robot xmlns:xacro="http://www.ros.org/wiki/xacro"
-       name="elmo_test_rig" >
+       name="rig1_rig2" >
   <xacro:include filename="$(find ipa_canopen_test)/urdf/elmo_test_rig.urdf.xacro" />
   <link name="world" />"
