Commit message: renamed ipa_canopen_test to canopen_test_utils

File: canopen_test_utils/urdf/elmo_test_rig.urdf.xacro (robot description, xacro)
@@ -4,5 +4,5 @@
   <xacro:include filename="$(find cob_description)/urdf/common.xacro" />
   <xacro:include filename="$(find cob_description)/urdf/materials.urdf.xacro" />
-  <xacro:include filename="$(find ipa_canopen_test)/urdf/elmo_test_rig.transmission.xacro" />
+  <xacro:include filename="$(find canopen_test_utils)/urdf/elmo_test_rig.transmission.xacro" />
   <property name="base_height" value="0.04" />
   <property name="base_radius" value="0.01" />

File: canopen_test_utils/urdf/rig1.urdf.xacro (robot description, xacro)
@@ -2,5 +2,5 @@
 <robot xmlns:xacro="http://www.ros.org/wiki/xacro"
        name="rig1" >
-  <xacro:include filename="$(find ipa_canopen_test)/urdf/elmo_test_rig.urdf.xacro" />
+  <xacro:include filename="$(find canopen_test_utils)/urdf/elmo_test_rig.urdf.xacro" />
   <link name="world" />"
   <xacro:elmo_test_rig prefix="rig1_" parent="world">

File: canopen_test_utils/urdf/rig12.urdf.xacro (robot description, xacro)
@@ -1,6 +1,6 @@
 <?xml version="1.0"?>
 <robot xmlns:xacro="http://www.ros.org/wiki/xacro"
-       name="rig1_rig2" >
-  <xacro:include filename="$(find ipa_canopen_test)/urdf/elmo_test_rig.urdf.xacro" />
+       name="rig12" >
+  <xacro:include filename="$(find canopen_test_utils)/urdf/elmo_test_rig.urdf.xacro" />
   <link name="world" />"
   <xacro:elmo_test_rig prefix="rig1_" parent="world">

File: canopen_test_utils/urdf/rig1_rig2.urdf.xacro (robot description, xacro)
@@ -1,9 +1,12 @@
 <?xml version="1.0"?>
 <robot xmlns:xacro="http://www.ros.org/wiki/xacro"
-       name="rig2" >
-  <xacro:include filename="$(find ipa_canopen_test)/urdf/elmo_test_rig.urdf.xacro" />
+       name="rig1_rig2" >
+  <xacro:include filename="$(find canopen_test_utils)/urdf/elmo_test_rig.urdf.xacro" />
   <link name="world" />"
+  <xacro:elmo_test_rig prefix="rig1_" parent="world">
+    <origin xyz="0.0 0.2 0.0" rpy="0 0 0" />
+  </xacro:elmo_test_rig>
   <xacro:elmo_test_rig prefix="rig2_" parent="world">
-    <origin xyz="0.0 0.0 0.0" rpy="0 0 0" />
+    <origin xyz="0.0 -0.2 0.0" rpy="0 0 0" />
   </xacro:elmo_test_rig>
   <gazebo>

File: canopen_test_utils/urdf/rig2.urdf.xacro (robot description, xacro)
@@ -1,12 +1,9 @@
 <?xml version="1.0"?>
 <robot xmlns:xacro="http://www.ros.org/wiki/xacro"
-       name="rig12" >
-  <xacro:include filename="$(find ipa_canopen_test)/urdf/elmo_test_rig.urdf.xacro" />
+       name="rig2" >
+  <xacro:include filename="$(find canopen_test_utils)/urdf/elmo_test_rig.urdf.xacro" />
   <link name="world" />"
-  <xacro:elmo_test_rig prefix="rig1_" parent="world">
-    <origin xyz="0.0 0.2 0.0" rpy="0 0 0" />
-  </xacro:elmo_test_rig>
   <xacro:elmo_test_rig prefix="rig2_" parent="world">
-    <origin xyz="0.0 -0.2 0.0" rpy="0 0 0" />
+    <origin xyz="0.0 0.0 0.0" rpy="0 0 0" />
   </xacro:elmo_test_rig>
   <gazebo>
